File: 65-keyboard-practice.kicad_pcb (KiCad board)
At the start: 2 copper layers, 311.2 x 133.4 mm, 140 parts, among them SW1 SW_MEC_5E, SW10 #8, SW11 #9, SW12 #0, SW13 -_, SW14 =+, SW15 BKSP, SW16 DEL, SW17 TAB, SW18 Q, SW19 W, SW2 Esc, SW20 E, SW21 R, SW22 T, SW23 Y, SW24 U, SW25 I, SW26 O, SW27 P, SW28 [{, SW29 ]}, SW3 #1, SW30 \|, SW31 HOME, SW32 CPLK, SW33 A, SW34 S, SW35 D, SW36 F, SW37 G, SW38 H, SW39 J, SW4 #2, SW40 K, SW41 L, SW42 ;:, SW43 '", SW44 ENTER, SW45 PGUP, SW46 LSHFT, SW47 Z, SW48 X, SW49 C, SW5 #3, SW50 V, SW51 B, SW52 N, SW53 M, SW54 ,<, SW55 .>, SW56 /?, SW57 RSHFT, SW58 UP, SW59 PGDN, SW6 #4, SW60 CTRL, SW61 WIN, SW62 LALT, SW63 SPACE, SW64 RALT, SW65 FN, SW66 FN2, SW67 LEFT, SW68 DOWN, SW69 RIGHT, SW7 #5, SW8 #6, SW9 #7, U1 ProMicro

Commit message: Finished provisional routing
Parts:
- moved D54 26.2 mm to (290.7, 76.9)
- moved D39 26.1 mm to (270.5, 74.8)
- moved D66 25.9 mm to (316.1, 77.0)
- moved D10 23.5 mm to (285.6, 70.4)
- moved D68 23.5 mm to (339.1, 79.2)
- moved D25 23.1 mm to (283.1, 72.6)
- moved D53 22.9 mm to (278.0, 76.9)
- moved D40 22.9 mm to (280.6, 74.8)
- moved D24 21.8 mm to (273.0, 72.6)
- moved D41 21.7 mm to (293.2, 74.7)
- moved D56 21.4 mm to (318.6, 74.8)
- moved D12 21.2 mm to (310.9, 70.4)
- moved D27 20.7 mm to (308.4, 72.6)
- moved D42 20.5 mm to (305.9, 74.7)
- moved D55 20.4 mm to (303.4, 76.9)
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Routing:
- net COL0: track 0.00 -> 349.2 mm, vias 0 -> 1
- net COL1: track 0.00 -> 343.1 mm, vias 0 -> 1
- net ROW0: track 0.00 -> 340.8 mm, vias 0 -> 1
- net ROW1: track 0.00 -> 328.0 mm, vias 0 -> 3
- net ROW2: track 0.00 -> 314.0 mm, vias 0 -> 1
- net ROW3: track 0.00 -> 313.9 mm, vias 0 -> 1
- net ROW4: track 0.00 -> 311.3 mm, vias 0 -> 3
- net COL6: track 0.00 -> 296.9 mm, vias 0 -> 1
- net COL5: track 0.00 -> 292.6 mm, vias 0 -> 1
- net COL2: track 0.00 -> 275.6 mm, vias 0 -> 1
- net COL7: track 0.00 -> 225.5 mm, vias 0 -> 1
- net COL4: track 0.00 -> 224.4 mm, vias 0 -> 1
- net COL3: track 0.00 -> 216.0 mm, vias 0 -> 1
- net Net-(D62-Pad2): track 0.00 -> 158.3 mm
- net Net-(D52-Pad2): track 0.00 -> 144.4 mm
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
Commit message: Some esthetic details
Parts:
- moved D10 13.6 mm to (299.2, 71.9)
- moved D9 13.6 mm to (289.0, 71.9)
- moved D25 13.6 mm to (296.6, 74.0)
- moved D40 13.6 mm to (294.1, 76.2)
- moved D53 13.6 mm to (291.5, 78.2)
- moved D54 13.6 mm to (304.2, 78.2)
- moved D24 13.5 mm to (286.5, 74.0)
- moved D41 13.5 mm to (306.7, 76.2)
- moved D39 13.5 mm to (283.9, 76.2)
- moved D63 13.5 mm to (301.7, 79.5)
- moved D26 13.5 mm to (309.2, 74.0)
- moved D11 13.5 mm to (311.7, 71.9)
- moved D12 13.4 mm to (324.3, 71.9)
- moved D27 13.4 mm to (321.7, 74.0)
- moved D42 13.4 mm to (319.2, 76.2)
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Routing:
- net COL2: track 275.6 -> 301.0 mm
- net ROW4: track 311.3 -> 324.5 mm
- net Net-(D53-Pad2): track 125.3 -> 137.7 mm
- net Net-(D9-Pad2): track 76.6 -> 88.9 mm
- net Net-(D27-Pad2): track 79.7 -> 91.9 mm
- net Net-(D57-Pad2): track 95.6 -> 107.7 mm
- net Net-(D42-Pad2): track 97.7 -> 109.8 mm
- net Net-(D63-Pad2): track 136.8 -> 148.9 mm
- net Net-(D54-Pad2): track 119.3 -> 131.3 mm
- net Net-(D41-Pad2): track 101.6 -> 113.5 mm
- net Net-(D67-Pad2): track 110.8 -> 122.7 mm
- net Net-(D24-Pad2): track 99.0 -> 110.8 mm
- net Net-(D43-Pad2): track 73.5 -> 85.3 mm
- net Net-(D66-Pad2): track 130.4 -> 141.9 mm
- net Net-(D39-Pad2): track 116.5 -> 128.0 mm
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Other:
- board text added: "Teckt68v0.2"
- board text removed: "Teckt68v0.1"

Commit message: Added mounting holes
Parts:
- added REF**: MountingHole_2.2mm_M2_Pad, cftkb:MountingHole_2.2mm_M2_Pad, F.Cu at (210.8, 90.6)
- added REF**: MountingHole_2.2mm_M2_Pad, cftkb:MountingHole_2.2mm_M2_Pad, F.Cu at (210.8, 186.5)
- added REF**: MountingHole_2.2mm_M2_Pad, cftkb:MountingHole_2.2mm_M2_Pad, F.Cu at (355.7, 71.9)
- added REF**: MountingHole_2.2mm_M2_Pad, cftkb:MountingHole_2.2mm_M2_Pad, F.Cu at (60.4, 186.6)
- added REF**: MountingHole_2.2mm_M2_Pad, cftkb:MountingHole_2.2mm_M2_Pad, F.Cu at (361.3, 90.6)
- added REF**: MountingHole_2.2mm_M2_Pad, cftkb:MountingHole_2.2mm_M2_Pad, F.Cu at (60.4, 90.6)
- added REF**: MountingHole_2.2mm_M2_Pad, cftkb:MountingHole_2.2mm_M2_Pad, F.Cu at (361.3, 186.6)
- added REF**: MountingHole_2.2mm_M2_Pad, cftkb:MountingHole_2.2mm_M2_Pad, F.Cu at (66.0, 71.9)
Routing:
- net Net-(D15-Pad2): track 34.0 -> 31.6 mm
- net ROW0: track 349.8 -> 351.9 mm
- net Net-(D45-Pad2): track 86.9 -> 88.5 mm
- net ROW1: track 336.4 -> 337.8 mm
- net Net-(D30-Pad2): track 50.7 -> 49.5 mm
- net ROW4: track 324.5 -> 323.5 mm
- net ROW2: track 324.8 -> 325.8 mm
